File: RGB-to-component-covers.kicad_pcb (KiCad board)
At the start: 2 copper layers, 58.9 x 150.6 mm, 22 parts

Commit message: covers gerb for vga/shart->component
Other:
- board text added: "RGB to YPbPr transcoder wakabavideo.com"
- board text removed: "YPbPr to RGB transcoder wakabavideo.com"

Commit message: covers updated
Other:
- net class Default removed
