File: RGB-to-component.kicad_sch (KiCad schematic)
At the start: 61 parts, among them J1 VGA, J3 USB_C_Receptacle_Power, J4 SCART_CONN, J5 3xRCA_CONN, U1 SC6206B-65K5, U10 74HC86, U2 TPF141-TR, U3 RS8752XK, U4 TPF141-TR, U5 TPF141-TR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

Commit message: remember to save the schematic too
Parts:
- U10: footprint Package_SO:SOIC-14_3.9x8.7mm_P1.27mm -> Package_SO:TSSOP-14_4.4x5mm_P0.65mm
Changed lines of the file:
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@@
 			)
 		)
-		(property "Footprint" "Package_SO:SOIC-14_3.9x8.7mm_P1.27mm"
+		(property "Footprint" "Package_SO:TSSOP-14_4.4x5mm_P0.65mm"
 			(at 260.35 149.86 0)
 			(effects
@@
 			)
 		)
-		(property "Footprint" "Package_SO:SOIC-14_3.9x8.7mm_P1.27mm"
+		(property "Footprint" "Package_SO:TSSOP-14_4.4x5mm_P0.65mm"
 			(at 99.06 85.09 0)
 			(effects
@@
 			)
 		)
-		(property "Footprint" "Package_SO:SOIC-14_3.9x8.7mm_P1.27mm"
+		(property "Footprint" "Package_SO:TSSOP-14_4.4x5mm_P0.65mm"
 			(at 83.82 82.55 0)
 			(effects
@@
 			)
 		)
-		(property "Footprint" "Package_SO:SOIC-14_3.9x8.7mm_P1.27mm"
+		(property "Footprint" "Package_SO:TSSOP-14_4.4x5mm_P0.65mm"
 			(at 110.49 109.22 0)
 			(effects
@@
 			)
 		)
-		(property "Footprint" "Package_SO:SOIC-14_3.9x8.7mm_P1.27mm"
+		(property "Footprint" "Package_SO:TSSOP-14_4.4x5mm_P0.65mm"
 			(at 236.22 142.24 0)
 			(effects

Commit message: change back to THS7374
Parts:
- removed U2, U4, U5, U9: TPF141-TR, Package_TO_SOT_SMD:SOT-23-6_Handsoldering, symbol videobits:TPF141-TR
- added U6: THS7374, Package_SO:TSSOP-14_4.4x5mm_P0.65mm, symbol Amplifier_Video:THS7374
- L101: value 10u -> 10uH
Connections:
- net 2B: now also U6.11 (CH4_OUT)
- net 2G: now also U6.12 (CH3_OUT)
- net 2R: now also U6.13 (CH2_OUT)
- net 2Y: now also U6.14 (CH1_OUT)
- net GND: now also U6.5 (GND), U6.6 (DISABLE)
- net VCC: now also U6.10 (V_{S+}), U6.9 (BYPASS)
- net at C1.1: now also U6.2 (CH2_IN)
- net at C2.1: now also U6.3 (CH3_IN)
- net at C3.1: now also U6.4 (CH4_IN)
- net at R20.1, R21.1, R22.1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: now also U6.1 (CH1_IN)

Commit message: swap to THS7374, updated parts
Parts:
- C5: LCSC C16133 -> C7171
- C7: LCSC C16133 -> C16133
- R10, R11, R15, R3, R4, R5, R9: LCSC C20638 -> C17820
- R13, R28: LCSC C40880 -> C101451
- R21: LCSC C273884 -> C17736
- R22: LCSC C26009 -> C322392
- U10: LCSC (none) -> C471866
- U6: LCSC (none) -> C2652746
Changed lines of the file:
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@@
 			)
 		)
-		(property "LCSC" "C20638"
+		(property "LCSC" "C17820"
 			(at 241.3 39.37 0)
 			(effects
@@
 			)
 		)
-		(property "LCSC" "C20638"
+		(property "LCSC" "C17820"
 			(at 236.22 44.45 0)
 			(effects
@@
 			)
 		)
-		(property "LCSC" "C20638"
+		(property "LCSC" "C17820"
 			(at 231.14 41.91 0)
 			(effects
@@
 			)
 		)
-		(property "LCSC" "C20638"
+		(property "LCSC" "C17820"
 			(at 129.54 59.69 0)
 			(effects
@@
 			)
 		)
-		(property "LCSC" "C20638"
+		(property "LCSC" "C17820"
 			(at 132.08 59.69 0)
 			(effects
@@
 			)
 		)
-		(property "LCSC" "C20638"
+		(property "LCSC" "C17820"
 			(at 134.62 59.69 0)
 			(effects
@@
 			)
 		)
-		(property "LCSC" " C16133"
+		(property "LCSC" "C16133"
 			(at 143.51 167.64 0)
 			(effects
@@
 			)
 		)
-		(property "LCSC" "C20638"
+		(property "LCSC" "C17820"
 			(at 31.75 118.11 0)
 			(effects
@@
 			)
 		)
-		(property "LCSC" "C273884"
+		(property "LCSC" "C17736"
 			(at 198.12 50.8 0)
 			(effects
@@
 			)
 		)
-		(property "LCSC" "C26009"
+		(property "LCSC" "C322392"
 			(at 198.12 53.34 0)
 			(effects
@@
 			)
 		)
-		(property "LCSC" "C40880"
+		(property "LCSC" "C101451"
 			(at 190.5 101.6 0)
 			(effects
@@
 			)
 		)
-		(property "LCSC" "C40880"
+		(property "LCSC" "C101451"
 			(at 254 104.14 0)
 			(effects
@@
 			)
 		)
-		(property "LCSC" " C16133"
+		(property "LCSC" "C7171"
 			(at 111.76 167.64 0)
 			(effects
@@
 			)
 		)
+		(property "LCSC" "C471866"
+			(at 98.7552 76.2 0)
+			(effects
+				(font
+					(size 1.27 1.27)
+				)
+				(hide yes)
+			)
+		)
 		(pin "5"
 		)
@@
 			)
 		)
+		(property "LCSC" "C471866"
+			(at 83.5152 73.66 0)
+			(effects
+				(font
+					(size 1.27 1.27)
+				)
+				(hide yes)
+			)
+		)
 		(pin "5"
 		)
@@
 			)
 		)
+		(property "LCSC" "C471866"
+			(at 110.1852 100.33 0)
+			(effects
+				(font
+					(size 1.27 1.27)
+				)
+				(hide yes)
+			)
+		)
 		(pin "5"
 		)
@@
 			)
 		)
+		(property "LCSC" "C2652746"
+			(at 166.0241 38.1 0)
+			(effects
+				(font
+					(size 1.27 1.27)
+				)
+				(hide yes)
+			)
+		)
 		(pin "3"
 		)
@@
 			(effects
 				(font
+					(size 1.27 1.27)
+				)
+				(hide yes)
+			)
+		)
+		(property "LCSC" "C471866"
+			(at 242.57 140.9699 0)
+			(effects
+				(font
